File: nRF52840_breakout.kicad_pcb (KiCad board)
At the start: 4 copper layers, 24.1 x 34.3 mm, 66 parts, among them J2 Conn_ARM_JTAG_SWD_10, J3 Conn_01x22, J4 Conn_01x16, J5 Conn_01x22, J6 S2B-PH-SM4-TB(LF)(SN), J7 Conn_Coaxial, U1 nRF52840, U2 BQ24072, U3 TPS63031, U4 BME680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

Commit message: kicad
Other:
- net class Default removed
- net class RF removed
- net class VBUS removed
- net class VDD_BAT removed
- net class VDD_H removed
- net class VDD_nRF removed
- net class custom removed
